Commit message: + Update not finished

File: urdf/g1_29dof_lock_waist.urdf (robot description, URDF)
Before this commit: robot g1_29dof_lock_waist, 40 links, 39 joints
Links:
- link left_rubber_hand: geometry collision box size=0.20 0.07 0.10; visual mesh filename=package://mocopi_ros2/urdf/meshes/left_rubber_hand.STL
- link right_rubber_hand: geometry collision box size=0.20 0.07 0.10; visual mesh filename=package://mocopi_ros2/urdf/meshes/right_rubber_hand.STL

Commit message: + Update Collision Model

File: urdf/g1_29dof_lock_waist.urdf (robot description, URDF)
Before this commit: robot g1_29dof_lock_waist, 40 links, 39 joints
Links:
- link head_link: geometry collision mesh filename=package://mocopi_ros2/urdf/meshes/head_link_collision_model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; visual mesh filename=package://mocopi_ros2/urdf/meshes/head_link.STL
- link left_ankle_pitch_link: geometry collision mesh filename=package://mocopi_ros2/urdf/meshes/left_ankle_pitch_link_col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; visual mesh filename=package://mocopi_ros2/urdf/meshes/left_ankle_pitch_link.STL
- link left_elbow_link: geometry collision mesh filename=package://mocopi_ros2/urdf/meshes/left_elbow_link_collision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; visual mesh filename=package://mocopi_ros2/urdf/meshes/left_elbow_link.STL
- link left_hip_pitch_link: geometry collision mesh filename=package://mocopi_ros2/urdf/meshes/left_hip_pitch_link_colli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; visual mesh filename=package://mocopi_ros2/urdf/meshes/left_hip_pitch_link.STL
- link left_hip_roll_link: geometry collision mesh filename=package://mocopi_ros2/urdf/meshes/left_hip_roll_link_collis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; visual mesh filename=package://mocopi_ros2/urdf/meshes/left_hip_roll_link.STL
- link left_hip_yaw_link: geometry collision mesh filename=package://mocopi_ros2/urdf/meshes/left_hip_yaw_link_collisi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; visual mesh filename=package://mocopi_ros2/urdf/meshes/left_hip_yaw_link.STL
- link left_knee_link: geometry collision mesh filename=package://mocopi_ros2/urdf/meshes/left_knee_link_collision_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; visual mesh filename=package://mocopi_ros2/urdf/meshes/left_knee_link.STL
- link left_rubber_hand: geometry collision mesh filename=package://mocopi_ros2/urdf/meshes/left_rubber_hand_collisio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; visual mesh filename=package://mocopi_ros2/urdf/meshes/left_rubber_hand.STL
- link left_shoulder_yaw_link: geometry collision mesh filename=package://mocopi_ros2/urdf/meshes/left_shoulder_yaw_link_co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; visual mesh filename=package://mocopi_ros2/urdf/meshes/left_shoulder_yaw_link.STL
- link left_wrist_pitch_link: geometry collision mesh filename=package://mocopi_ros2/urdf/meshes/left_wrist_pitch_link_col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; visual mesh filename=package://mocopi_ros2/urdf/meshes/left_wrist_pitch_link.STL
- link left_wrist_roll_link: geometry collision mesh filename=package://mocopi_ros2/urdf/meshes/left_wrist_roll_link_coll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; visual mesh filename=package://mocopi_ros2/urdf/meshes/left_wrist_roll_link.STL
- link left_wrist_yaw_link: geometry collision mesh filename=package://mocopi_ros2/urdf/meshes/left_wrist_yaw_link_colli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; visual mesh filename=package://mocopi_ros2/urdf/meshes/left_wrist_yaw_link.STL
- link logo_link: geometry collision mesh filename=package://mocopi_ros2/urdf/meshes/logo_link_collision_model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; visual mesh filename=package://mocopi_ros2/urdf/meshes/logo_link.STL
- link pelvis_contour_link: geometry collision mesh filename=package://mocopi_ros2/urdf/meshes/pelvis_contour_link_colli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; visual mesh filename=package://mocopi_ros2/urdf/meshes/pelvis_contour_link.STL
- link right_ankle_pitch_link: geometry collision mesh filename=package://mocopi_ros2/urdf/meshes/right_ankle_pitch_link_co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; visual mesh filename=package://mocopi_ros2/urdf/meshes/right_ankle_pitch_link.STL
- link right_elbow_link: geometry collision mesh filename=package://mocopi_ros2/urdf/meshes/right_elbow_link_collisio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; visual mesh filename=package://mocopi_ros2/urdf/meshes/right_elbow_link.STL
- link right_hip_pitch_link: geometry collision mesh filename=package://mocopi_ros2/urdf/meshes/right_hip_pitch_link_coll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; visual mesh filename=package://mocopi_ros2/urdf/meshes/right_hip_pitch_link.STL
- link right_hip_roll_link: geometry collision mesh filename=package://mocopi_ros2/urdf/meshes/right_hip_roll_link_colli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; visual mesh filename=package://mocopi_ros2/urdf/meshes/right_hip_roll_link.STL
- link right_hip_yaw_link: geometry collision mesh filename=package://mocopi_ros2/urdf/meshes/right_hip_yaw_link_collis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; visual mesh filename=package://mocopi_ros2/urdf/meshes/right_hip_yaw_link.STL
- link right_knee_link: geometry collision mesh filename=package://mocopi_ros2/urdf/meshes/right_knee_link_collision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; visual mesh filename=package://mocopi_ros2/urdf/meshes/right_knee_link.STL
- link right_rubber_hand: geometry collision mesh filename=package://mocopi_ros2/urdf/meshes/right_rubber_hand_collisi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; visual mesh filename=package://mocopi_ros2/urdf/meshes/right_rubber_hand.STL
- link right_shoulder_yaw_link: geometry collision mesh filename=package://mocopi_ros2/urdf/meshes/right_shoulder_yaw_link_c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; visual mesh filename=package://mocopi_ros2/urdf/meshes/right_shoulder_yaw_link.S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
- link right_wrist_pitch_link: geometry collision mesh filename=package://mocopi_ros2/urdf/meshes/right_wrist_pitch_link_co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; visual mesh filename=package://mocopi_ros2/urdf/meshes/right_wrist_pitch_link.STL
- link right_wrist_roll_link: geometry collision mesh filename=package://mocopi_ros2/urdf/meshes/right_wrist_roll_link_col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; visual mesh filename=package://mocopi_ros2/urdf/meshes/right_wrist_roll_link.STL
- link right_wrist_yaw_link: geometry collision mesh filename=package://mocopi_ros2/urdf/meshes/right_wrist_yaw_link_coll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; visual mesh filename=package://mocopi_ros2/urdf/meshes/right_wrist_yaw_link.STL
- link torso_link: geometry collision mesh filename=package://mocopi_ros2/urdf/meshes/torso_link_collision_mode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; visual mesh filename=package://mocopi_ros2/urdf/meshes/torso_link.STL
- link waist_support_link: geometry collision mesh filename=package://mocopi_ros2/urdf/meshes/waist_support_link_collis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; visual mesh filename=package://mocopi_ros2/urdf/meshes/waist_support_link.STL
